File: AP3429-tryout.sch (KiCad schematic (older format))
At the start: 25 parts, among them U1 AP3429, U2 AP3429, U3 AP3429, U4 AP2120N

Commit message: update,
Parts:
- removed L1, L2, L3: L_2.2uH_CD43, symbol taobao-l:L_2.2uH_CD43
- added H1, H2, H3, H4: MOUNT_M3, MountingHole:MountingHole_3.2mm_M3_DIN965, symbol taobao-mounting-hole:MOUNT_M3
- added L1, L2, L3: L_2.2uH,CD43, w_smd_inductors:inductor_smd_4.8x2.8mm, symbol taobao-l:L_2.2uH,CD43
- D1: footprint (none) -> LED_SMD:LED_0805_2012Metric_Castellated
- U4: footprint (none) -> Package_TO_SOT_SMD:SOT-23_Handsoldering
- gave numbers to parts that had none: 10
Changed lines of the file:
@@
 	2500 1300 1950 1300
-$Comp
-L taobao-l:L_2.2uH_CD43 L1
-U 1 1 5C039135
-P 4700 1300
-F 0 "L1" V 4885 1300 50  0000 C CNN
-F 1 "L_2.2uH_CD43" V 4794 1300 50  0000 C CNN
-F 2 "" H 4700 1300 50  0001 C CNN
-F 3 "~" H 4700 1300 50  0001 C CNN
-	1    4700 1300
-	0    -1   -1   0
-$EndComp
 $Comp
 L taobao-r:R304,0603 R1
@@
 	2500 3450 1950 3450
 $Comp
-L taobao-l:L_2.2uH_CD43 L2
-U 1 1 5C03B21E
-P 4700 3450
-F 0 "L2" V 4885 3450 50  0000 C CNN
-F 1 "L_2.2uH_CD43" V 4794 3450 50  0000 C CNN
-F 2 "" H 4700 3450 50  0001 C CNN
-F 3 "~" H 4700 3450 50  0001 C CNN
-	1    4700 3450
-	0    -1   -1   0
-$EndComp
-$Comp
 L taobao-r:R304,0603 R3
 U 1 1 5C03B22A
@@
 Wire Wire Line
 	2500 5750 1950 5750
-$Comp
-L taobao-l:L_2.2uH_CD43 L3
-U 1 1 5C03BF1C
-P 4700 5750
-F 0 "L3" V 4885 5750 50  0000 C CNN
-F 1 "L_2.2uH_CD43" V 4794 5750 50  0000 C CNN
-F 2 "" H 4700 5750 50  0001 C CNN
-F 3 "~" H 4700 5750 50  0001 C CNN
-	1    4700 5750
-	0    -1   -1   0
-$EndComp
 Wire Wire Line
 	4200 5750 4600 5750
@@
 F 0 "D1" V 6296 6382 50  0000 R CNN
 F 1 "LED_ORANGE" V 6205 6382 50  0000 R CNN
-F 2 "" V 6250 6450 50  0001 C CNN
+F 2 "LED_SMD:LED_0805_2012Metric_Castellated" V 6250 6450 50  0001 C CNN
 F 3 "~" V 6250 6450 50  0001 C CNN
 	1    6250 6450
@@
 	6250 6850 5600 6850
 $Comp
-L taobao-components:AP2120N U4
-U 1 1 5C048104
-P 9000 1950
-F 0 "U4" H 9000 2515 50  0000 C CNN
-F 1 "AP2120N" H 9000 2424 50  0000 C CNN
-F 2 "" H 9000 1950 50  0001 C CNN
-F 3 "" H 9000 1950 50  0001 C CNN
-	1    9000 1950
-	1    0    0    -1
-$EndComp
-$Comp
 L power:+3V3 #PWR0110
 U 1 1 5C0481CC
@@
 $EndComp
 $Comp
-L taobao-c:C226-6.3v,0603 C?
+L taobao-c:C226-6.3v,0603 C1
 U 1 1 5C061252
 P 1950 1850
-F 0 "C?" H 2042 1896 50  0000 L CNN
+F 0 "C1" H 2042 1896 50  0000 L CNN
 F 1 "C226-6.3v,0603" H 2042 1805 50  0000 L CNN
 F 2 "Capacitor_SMD:C_0603_1608Metric_Pad1.05x0.95mm_HandSolder" H 1950 1850 50  0001 C CNN
@@
 $EndComp
 $Comp
-L taobao-c:C226-6.3v,0603 C?
+L taobao-c:C226-6.3v,0603 C7
 U 1 1 5C0615D3
 P 6500 1650
-F 0 "C?" H 6592 1696 50  0000 L CNN
+F 0 "C7" H 6592 1696 50  0000 L CNN
 F 1 "C226-6.3v,0603" H 6592 1605 50  0000 L CNN
 F 2 "Capacitor_SMD:C_0603_1608Metric_Pad1.05x0.95mm_HandSolder" H 6500 1650 50  0001 C CNN
@@
 $EndComp
 $Comp
-L taobao-c:C226-6.3v,0603 C?
+L taobao-c:C226-6.3v,0603 C2
 U 1 1 5C061987
 P 1950 4000
-F 0 "C?" H 2042 4046 50  0000 L CNN
+F 0 "C2" H 2042 4046 50  0000 L CNN
 F 1 "C226-6.3v,0603" H 2042 3955 50  0000 L CNN
 F 2 "Capacitor_SMD:C_0603_1608Metric_Pad1.05x0.95mm_HandSolder" H 1950 4000 50  0001 C CNN
@@
 $EndComp
 $Comp
-L taobao-c:C226-6.3v,0603 C?
+L taobao-c:C226-6.3v,0603 C8
 U 1 1 5C0619F3
 P 6500 3800
-F 0 "C?" H 6592 3846 50  0000 L CNN
+F 0 "C8" H 6592 3846 50  0000 L CNN
 F 1 "C226-6.3v,0603" H 6592 3755 50  0000 L CNN
 F 2 "Capacitor_SMD:C_0603_1608Metric_Pad1.05x0.95mm_HandSolder" H 6500 3800 50  0001 C CNN
@@
 $EndComp
 $Comp
-L taobao-c:C226-6.3v,0603 C?
+L taobao-c:C226-6.3v,0603 C9
 U 1 1 5C061AE8
 P 6500 6100
-F 0 "C?" H 6592 6146 50  0000 L CNN
+F 0 "C9" H 6592 6146 50  0000 L CNN
 F 1 "C226-6.3v,0603" H 6592 6055 50  0000 L CNN
 F 2 "Capacitor_SMD:C_0603_1608Metric_Pad1.05x0.95mm_HandSolder" H 6500 6100 50  0001 C CNN
@@
 $EndComp
 $Comp
-L taobao-c:C226-6.3v,0603 C?
+L taobao-c:C226-6.3v,0603 C3
 U 1 1 5C061B56
 P 1950 6350
-F 0 "C?" H 2042 6396 50  0000 L CNN
+F 0 "C3" H 2042 6396 50  0000 L CNN
 F 1 "C226-6.3v,0603" H 2042 6305 50  0000 L CNN
 F 2 "Capacitor_SMD:C_0603_1608Metric_Pad1.05x0.95mm_HandSolder" H 1950 6350 50  0001 C CNN
@@
 $EndComp
 $Comp
-L taobao-c:C22pf,0603 C?
+L taobao-c:C22pf,0603 C6
 U 1 1 5C061E10
 P 5150 6000
-F 0 "C?" H 5242 6046 50  0000 L CNN
+F 0 "C6" H 5242 6046 50  0000 L CNN
 F 1 "C22pf,0603" H 5242 5955 50  0000 L CNN
 F 2 "Capacitor_SMD:C_0603_1608Metric_Pad1.05x0.95mm_HandSolder" H 5150 6000 50  0001 C CNN
@@
 $EndComp
 $Comp
-L taobao-c:C22pf,0603 C?
+L taobao-c:C22pf,0603 C5
 U 1 1 5C0621B0
 P 5150 3700
-F 0 "C?" H 5242 3746 50  0000 L CNN
+F 0 "C5" H 5242 3746 50  0000 L CNN
 F 1 "C22pf,0603" H 5242 3655 50  0000 L CNN
 F 2 "Capacitor_SMD:C_0603_1608Metric_Pad1.05x0.95mm_HandSolder" H 5150 3700 50  0001 C CNN
@@
 $EndComp
 $Comp
-L taobao-c:C22pf,0603 C?
+L taobao-c:C22pf,0603 C4
 U 1 1 5C06221C
 P 5150 1550
-F 0 "C?" H 5242 1596 50  0000 L CNN
+F 0 "C4" H 5242 1596 50  0000 L CNN
 F 1 "C22pf,0603" H 5242 1505 50  0000 L CNN
 F 2 "Capacitor_SMD:C_0603_1608Metric_Pad1.05x0.95mm_HandSolder" H 5150 1550 50  0001 C CNN
@@
 $EndComp
 $Comp
-L taobao-c:C106,0603 C?
+L taobao-c:C106,0603 C10
 U 1 1 5C0629A0
 P 9900 1950
-F 0 "C?" H 9992 1996 50  0000 L CNN
+F 0 "C10" H 9992 1996 50  0000 L CNN
 F 1 "C106,0603" H 9992 1905 50  0000 L CNN
 F 2 "Capacitor_SMD:C_0603_1608Metric_Pad1.05x0.95mm_HandSolder" H 9900 1950 50  0001 C CNN
@@
 	1    0    0    -1
 $EndComp
+$Comp
+L taobao-l:L_2.2uH,CD43 L1
+U 1 1 5C06343C
+P 4700 1300
+F 0 "L1" V 4885 1300 50  0000 C CNN
+F 1 "L_2.2uH,CD43" V 4794 1300 50  0000 C CNN
+F 2 "w_smd_inductors:inductor_smd_4.8x2.8mm" H 4700 1300 50  0001 C CNN
+F 3 "" H 4700 1300 50  0001 C CNN
+	1    4700 1300
+	0    -1   -1   0
+$EndComp
+$Comp
+L taobao-l:L_2.2uH,CD43 L2
+U 1 1 5C063614
+P 4700 3450
+F 0 "L2" V 4885 3450 50  0000 C CNN
+F 1 "L_2.2uH,CD43" V 4794 3450 50  0000 C CNN
+F 2 "w_smd_inductors:inductor_smd_4.8x2.8mm" H 4700 3450 50  0001 C CNN
+F 3 "" H 4700 3450 50  0001 C CNN
+	1    4700 3450
+	0    -1   -1   0
+$EndComp
+$Comp
+L taobao-l:L_2.2uH,CD43 L3
+U 1 1 5C0638E1
+P 4700 5750
+F 0 "L3" V 4885 5750 50  0000 C CNN
+F 1 "L_2.2uH,CD43" V 4794 5750 50  0000 C CNN
+F 2 "w_smd_inductors:inductor_smd_4.8x2.8mm" H 4700 5750 50  0001 C CNN
+F 3 "" H 4700 5750 50  0001 C CNN
+	1    4700 5750
+	0    -1   -1   0
+$EndComp
+$Comp
+L taobao-components:AP2120N U4
+U 1 1 5C066287
+P 9000 1950
+F 0 "U4" H 9000 2515 50  0000 C CNN
+F 1 "AP2120N" H 9000 2424 50  0000 C CNN
+F 2 "Package_TO_SOT_SMD:SOT-23_Handsoldering" H 8900 1450 50  0001 C CNN
+F 3 "" H 9000 1950 50  0001 C CNN
+	1    9000 1950
+	1    0    0    -1
+$EndComp
+$Comp
+L taobao-mounting-hole:MOUNT_M3 H1
+U 1 1 5C066ADD
+P 9100 5600
+F 0 "H1" H 9200 5646 50  0000 L CNN
+F 1 "MOUNT_M3" H 9200 5555 50  0000 L CNN
+F 2 "MountingHole:MountingHole_3.2mm_M3_DIN965" H 9100 5600 50  0001 C CNN
+F 3 "~" H 9100 5600 50  0001 C CNN
+	1    9100 5600
+	1    0    0    -1
+$EndComp
+$Comp
+L taobao-mounting-hole:MOUNT_M3 H2
+U 1 1 5C066BE5
+P 9550 5600
+F 0 "H2" H 9650 5646 50  0000 L CNN
+F 1 "MOUNT_M3" H 9650 5555 50  0000 L CNN
+F 2 "MountingHole:MountingHole_3.2mm_M3_DIN965" H 9550 5600 50  0001 C CNN
+F 3 "~" H 9550 5600 50  0001 C CNN
+	1    9550 5600
+	1    0    0    -1
+$EndComp
+$Comp
+L taobao-mounting-hole:MOUNT_M3 H3
+U 1 1 5C066C39
+P 9950 5600
+F 0 "H3" H 10050 5646 50  0000 L CNN
+F 1 "MOUNT_M3" H 10050 5555 50  0000 L CNN
+F 2 "MountingHole:MountingHole_3.2mm_M3_DIN965" H 9950 5600 50  0001 C CNN
+F 3 "~" H 9950 5600 50  0001 C CNN
+	1    9950 5600
+	1    0    0    -1
+$EndComp
+$Comp
+L taobao-mounting-hole:MOUNT_M3 H4
+U 1 1 5C066C8D
+P 10350 5600
+F 0 "H4" H 10450 5646 50  0000 L CNN
+F 1 "MOUNT_M3" H 10450 5555 50  0000 L CNN
+F 2 "MountingHole:MountingHole_3.2mm_M3_DIN965" H 10350 5600 50  0001 C CNN
+F 3 "~" H 10350 5600 50  0001 C CNN
+	1    10350 5600
+	1    0    0    -1
+$EndComp
