File: AP3429-tryout.kicad_pcb (KiCad board)
At the start: 2 copper layers, 90 x 50 mm, 29 parts, among them U1 AP3429, U2 AP3429, U3 AP3429, U4 AP2120N

Commit message: update,
Parts:
- added J1: Conn_01x05, Connector_PinHeader_2.54mm:PinHeader_1x05_P2.54mm_Vertical, F.Cu at (4.69, 12.4)
- added J2: Conn_01x02, Connector_PinHeader_2.54mm:PinHeader_1x02_P2.54mm_Vertical, F.Cu at (4.69, 2.98)
- C1, C2, C3, C7, C8, C9: value C226-6.3v,0603 -> C226,6.3v,0603
- D1: footprint LED_SMD:LED_0603_1608Metric_Pad1.05x0.95mm_HandSolder -> LED_SMD:LED_0805_2012Metric_Castellated
- moved R6 100.7 mm to (46.4, 41.3), turned to 90 degrees
- moved C9 98.7 mm to (44.1, 45.4)
- moved R1 98.6 mm to (40.3, 10.2), turned to 180 degrees
- moved C10 98.6 mm to (58.4, 12.5), turned to 180 degrees
- moved R2 97.2 mm to (45.5, 8.94), turned to 270 degrees
- moved C6 96.0 mm to (40.6, 39.4), turned to 180 degrees
- moved L3 95.8 mm to (33.0, 34.7), turned to 90 degrees
- moved R5 93.1 mm to (40.5, 42.9), turned to 180 degrees
- moved R4 92.2 mm to (46.4, 25.5), turned to 270 degrees
- moved R3 91.0 mm to (40.9, 26.1), turned to 180 degrees
- moved C8 90.6 mm to (43.0, 29.9)
- moved L1 88.4 mm to (31.1, 6.55), turned to 90 degrees
- moved U4 87.8 mm to (58.4, 7.28), turned to 90 degrees
- moved L2 87.2 mm to (32.9, 22.9), turned to 90 degrees
- moved C3 85.6 mm to (25.0, 42.2)
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
Commit message: update,
Routing:
- net GND: track 0.00 -> 188.7 mm
- net +3V3: track 0.00 -> 123.9 mm
- net +5V: track 0.00 -> 72.6 mm
- net +3V0: track 0.00 -> 63.8 mm, vias 0 -> 1
- net +1V2: track 0.00 -> 60.8 mm
- net +1V8: track 0.00 -> 49.4 mm, vias 0 -> 1
- net Net-(C6-Pad2): track 0.00 -> 45.4 mm
- net Net-(C4-Pad2): track 0.00 -> 34.9 mm
- net Net-(C5-Pad2): track 0.00 -> 31.3 mm
- net Net-(L1-Pad1): track 0.00 -> 9.30 mm
- net Net-(L2-Pad1): track 0.00 -> 8.45 mm
- net Net-(L3-Pad1): track 0.00 -> 7.24 mm
- net Net-(D1-Pad2): track 0.00 -> 2.92 mm

Commit message: update,
Parts:
- added C11: C104,0603, Capacitor_SMD:C_0603_1608Metric_Pad1.05x0.95mm_HandSolder, F.Cu at (60.6, 5.40)
- added C12: C104,0603, Capacitor_SMD:C_0603_1608Metric_Pad1.05x0.95mm_HandSolder, F.Cu at (67.2, 12.5)
- added C13: C104,0603, Capacitor_SMD:C_0603_1608Metric_Pad1.05x0.95mm_HandSolder, F.Cu at (48.4, 13.3)
- added C14: CP47uf,10V, w_smd_cap:c_elec_5x5.3, F.Cu at (56.7, 6.40)
- added C15: C104,0603, Capacitor_SMD:C_0603_1608Metric_Pad1.05x0.95mm_HandSolder, F.Cu at (79.9, 3.50)
- added C16: CP47uf,10V, w_smd_cap:c_elec_5x5.3, F.Cu at (75.9, 5.60)
- added C17: C104,0603, Capacitor_SMD:C_0603_1608Metric_Pad1.05x0.95mm_HandSolder, F.Cu at (48.3, 28.5)
- added C18: C104,0603, Capacitor_SMD:C_0603_1608Metric_Pad1.05x0.95mm_HandSolder, F.Cu at (60.5, 19.8)
- added C19: CP47uf,10V, w_smd_cap:c_elec_5x5.3, F.Cu at (56.9, 21.7)
- added C20: C104,0603, Capacitor_SMD:C_0603_1608Metric_Pad1.05x0.95mm_HandSolder, F.Cu at (67.2, 26.7)
- added C21: C104,0603, Capacitor_SMD:C_0603_1608Metric_Pad1.05x0.95mm_HandSolder, F.Cu at (80.4, 18.6)
- added C22: CP47uf,10V, w_smd_cap:c_elec_5x5.3, F.Cu at (75.6, 20.1)
- added C23: C104,0603, Capacitor_SMD:C_0603_1608Metric_Pad1.05x0.95mm_HandSolder, F.Cu at (48.4, 43.6)
- added C24: C104,0603, Capacitor_SMD:C_0603_1608Metric_Pad1.05x0.95mm_HandSolder, F.Cu at (61.0, 34.7)
- added C25: CP47uf,10V, w_smd_cap:c_elec_5x5.3, F.Cu at (56.9, 36.7)
- added C26: C104,0603, Capacitor_SMD:C_0603_1608Metric_Pad1.05x0.95mm_HandSolder, F.Cu at (67.7, 41.0)
- added C27: C104,0603, Capacitor_SMD:C_0603_1608Metric_Pad1.05x0.95mm_HandSolder, F.Cu at (80.5, 32.3)
- added C28: CP47uf,10V, w_smd_cap:c_elec_5x5.3, F.Cu at (76.3, 34.3)
- added TP1: TestPoint, TestPoint:TestPoint_Keystone_5019_Minature, F.Cu at (76.7, 12.5)
- added TP2: TestPoint, TestPoint:TestPoint_Keystone_5019_Minature, F.Cu at (58.4, 13.1)
- added TP3: TestPoint, TestPoint:TestPoint_Keystone_5019_Minature, F.Cu at (59.9, 27.9)
- added TP4: TestPoint, TestPoint:TestPoint_Keystone_5019_Minature, F.Cu at (79.3, 25.2)
- added TP5: TestPoint, TestPoint:TestPoint_Keystone_5019_Minature, F.Cu at (59.1, 43.3)
- added TP6: TestPoint, TestPoint:TestPoint_Keystone_5019_Minature, F.Cu at (77.1, 40.7)
- added U10: AMS1117-3.3, Package_TO_SOT_SMD:SOT-223-3_TabPin2, F.Cu at (69.6, 35.0)
- added U5: AMS1117-3.3, Package_TO_SOT_SMD:SOT-223-3_TabPin2, F.Cu at (69.1, 6.20)
- added U6: AMS1117-3.3, Package_TO_SOT_SMD:SOT-223-3_TabPin2, F.Cu at (50.0, 7.60)
- added U7: AMS1117-3.3, Package_TO_SOT_SMD:SOT-223-3_TabPin2, F.Cu at (50.2, 22.3)
- added U8: AMS1117-3.3, Package_TO_SOT_SMD:SOT-223-3_TabPin2, F.Cu at (69.1, 20.7)
- added U9: AMS1117-3.3, Package_TO_SOT_SMD:SOT-223-3_TabPin2, F.Cu at (50.1, 37.1)
- moved H1 37.8 mm to (115.6, 44.1)
- moved H2 37.8 mm to (121.7, 38.0)
- moved H3 37.8 mm to (121.7, 44.1)
- moved H4 37.8 mm to (115.6, 38.0)
- moved C10 19.0 mm to (39.4, 11.2)
- moved U4 19.0 mm to (39.4, 5.98)
- moved C7 13.6 mm to (30.9, 11.9)
- moved U1 13.1 mm to (11.9, 5.65)
- moved C3 11.9 mm to (13.3, 44.5)
- moved U3 11.7 mm to (13.8, 38.6)
- moved U2 11.6 mm to (14.3, 23.2)
- moved C1 11.4 mm to (12.2, 12.2)
- moved C2 11.4 mm to (13.3, 28.8)
- moved R1 11.4 mm to (29.2, 7.66)
- moved R2 11.4 mm to (34.4, 6.44)
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Routing:
- net +5V: track 72.6 -> 251.3 mm, vias 0 -> 3
- net GND: track 188.7 -> 355.9 mm, vias 0 -> 3
- net Net-(C15-Pad1): track 0.00 -> 27.4 mm
- net Net-(C24-Pad1): track 0.00 -> 26.7 mm
- net Net-(C27-Pad1): track 0.00 -> 25.9 mm
- net Net-(C18-Pad1): track 0.00 -> 25.6 mm
- net Net-(C21-Pad1): track 0.00 -> 24.7 mm
- net Net-(C11-Pad1): track 0.00 -> 24.5 mm
- net +1V2: track 60.8 -> 39.1 mm, vias 0 -> 1
- net Net-(C5-Pad2): track 31.3 -> 37.8 mm
- net Net-(C6-Pad2): track 45.4 -> 39.0 mm, vias 0 -> 2
- net Net-(D1-Pad2): track 2.92 -> 7.91 mm
- net Net-(C4-Pad2): track 34.9 -> 30.2 mm
- net +3V3: track 123.9 -> 120.4 mm, vias 0 -> 2
- net +1V8: track 49.4 -> 47.3 mm
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Other:
- net class Default: trace_width 0.25 -> 0.5; via_dia 0.8 -> 1.5
- net class GND added: clearance 0.2, trace_width 1, via_dia 1.5, via_drill 0.4
- net class PWR added: clearance 0.2, trace_width 0.75, via_dia 1.5, via_drill 0.4

Commit message: update,
Parts:
- C12, C18, C20: footprint Capacitor_SMD:C_0603_1608Metric_Pad1.05x0.95mm_HandSolder -> w_smd_cap:c_elec_5x5.3
- C14, C16, C19, C22, C25, C28: value CP47uf,10V -> CP47uf,50V; footprint w_smd_cap:c_elec_5x5.3 -> w_smd_cap:c_elec_6.3x7.7
- L1, L2, L3: value L_2.2uH,CD43 -> L_2.2uH,1210; footprint w_smd_inductors:inductor_smd_4.8x2.8mm -> Inductor_SMD:L_1210_3225Metric_Pad1.42x2.65mm_HandSolder
- turned L1 to 0 degrees
- turned L2 to 0 degrees
- turned L3 to 180 degrees

Commit message: update,
Parts:
- C12, C18, C20: footprint w_smd_cap:c_elec_5x5.3 -> Capacitor_SMD:C_0603_1608Metric_Pad1.05x0.95mm_HandSolder
- turned L3 to 0 degrees
- turned R5 to 0 degrees
Routing:
- net +5V: track 251.3 -> 315.1 mm
- net +3V0: track 64.3 -> 44.7 mm
- net GND: track 355.9 -> 367.9 mm, vias 3 -> 2
- net +3V3: track 120.4 -> 131.8 mm, vias 2 -> 1
- net +1V8: track 47.3 -> 54.7 mm
- net Net-(C5-Pad2): track 37.8 -> 43.7 mm
- net Net-(C6-Pad2): track 39.0 -> 33.7 mm
- net Net-(D1-Pad2): track 7.91 -> 2.85 mm
- net Net-(C24-Pad1): track 26.7 -> 23.7 mm
- net Net-(C27-Pad1): track 25.9 -> 27.0 mm
- net Net-(C4-Pad2): track 30.2 -> 30.9 mm
- net Net-(C21-Pad1): track 24.7 -> 25.4 mm
Other:
- net class Default: clearance 0.2 -> 0.5
- net class GND: clearance 0.2 -> 0.5
- net class PWR: clearance 0.2 -> 0.5
- rule trace_clearance: 0.2 -> 0.5

Commit message: update,
Parts:
- moved H4 115.4 mm to (5.00, 5.00)
- moved H1 113.6 mm to (5.00, 70.0)
- moved H2 49.4 mm to (85.0, 5.00)
- moved H3 44.9 mm to (85.0, 70.0)
- moved C19 13.3 mm to (59.9, 34.7)
- moved C20 13.3 mm to (70.2, 39.7)
- moved D1 13.3 mm to (9.30, 41.7)
- moved L2 13.3 mm to (27.7, 32.4)
- moved TP4 13.3 mm to (82.3, 38.2)
- moved U8 13.3 mm to (72.1, 33.7)
- moved C16 13.3 mm to (78.9, 18.6)
- moved TP2 13.3 mm to (61.4, 26.1)
- moved U6 13.3 mm to (53.0, 20.6)
- moved C1 13.3 mm to (15.2, 25.2)
- moved C10 13.3 mm to (42.4, 24.2)
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Routing:
- net +5V: track 315.1 -> 320.6 mm
- net GND: track 367.9 -> 372.4 mm
Other:
- board size 90 x 50 mm -> 90 x 75 mm

Commit message: update,
Parts:
- moved TP4 6.42 mm to (78.4, 43.3)
- moved C27 4.74 mm to (83.4, 50.0)
- moved TP6 4.65 mm to (78.4, 58.0)
- moved C15 4.15 mm to (83.4, 20.6)
- moved TP3 3.92 mm to (59.8, 43.3)
- moved C21 3.73 mm to (83.4, 35.3)
- moved TP1 3.36 mm to (78.4, 28.6)
- moved C26 3.05 mm to (70.4, 57.0)
- moved U10 2.97 mm to (70.4, 50.0)
- moved TP2 2.97 mm to (59.8, 28.6)
- moved C28 2.87 mm to (78.4, 50.0)
- moved TP5 2.87 mm to (59.8, 58.0)
- moved C18 2.85 mm to (64.8, 35.3)
- moved C20 2.64 mm to (70.4, 42.3)
- moved C11 2.52 mm to (64.8, 20.6)
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Routing:
- net GND: track 372.4 -> 0.00 mm, vias 2 -> 0
- net +5V: track 320.6 -> 0.00 mm, vias 3 -> 0
- net +3V3: track 131.8 -> 0.00 mm, vias 1 -> 0
- net +1V8: track 54.7 -> 0.00 mm, vias 1 -> 0
- net +3V0: track 44.7 -> 0.00 mm, vias 1 -> 0
- net Net-(C5-Pad2): track 43.7 -> 0.00 mm
- net +1V2: track 39.3 -> 0.00 mm, vias 1 -> 0
- net Net-(C6-Pad2): track 33.7 -> 0.00 mm, vias 2 -> 0
- net Net-(C4-Pad2): track 30.9 -> 0.00 mm
- net Net-(C15-Pad1): track 27.4 -> 0.00 mm
- net Net-(C27-Pad1): track 27.0 -> 0.00 mm
- net Net-(C18-Pad1): track 25.6 -> 0.00 mm
- net Net-(C21-Pad1): track 25.4 -> 0.00 mm
- net Net-(C11-Pad1): track 24.5 -> 0.00 mm
- net Net-(C24-Pad1): track 23.7 -> 0.00 mm
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
Commit message: update,
Parts:
- moved C15 8.00 mm to (75.4, 20.6)
- moved C21 8.00 mm to (75.4, 35.3)
- moved C27 8.00 mm to (75.4, 50.0)
- moved C11 8.00 mm to (56.8, 20.6)
- moved C18 8.00 mm to (56.8, 35.3)
- moved C24 8.00 mm to (56.8, 50.0)
Routing:
- net GND: track 0.00 -> 395.1 mm, vias 0 -> 2
- net +5V: track 0.00 -> 287.3 mm, vias 0 -> 5
- net +3V3: track 0.00 -> 111.5 mm, vias 0 -> 2
- net +3V0: track 0.00 -> 59.4 mm, vias 0 -> 1
- net +1V8: track 0.00 -> 43.7 mm, vias 0 -> 1
- net +1V2: track 0.00 -> 36.0 mm, vias 0 -> 1
- net Net-(C5-Pad2): track 0.00 -> 35.5 mm
- net Net-(C6-Pad2): track 0.00 -> 35.4 mm
- net Net-(C15-Pad1): track 0.00 -> 32.8 mm
- net Net-(C4-Pad2): track 0.00 -> 27.7 mm
- net Net-(C18-Pad1): track 0.00 -> 22.0 mm
- net Net-(C24-Pad1): track 0.00 -> 22.0 mm
- net Net-(C21-Pad1): track 0.00 -> 21.9 mm
- net Net-(C11-Pad1): track 0.00 -> 21.9 mm
- net Net-(C27-Pad1): track 0.00 -> 21.9 mm
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Other:
- net class Default: clearance 0.5 -> 0.2; trace_width 0.5 -> 0.3
- net class GND: clearance 0.5 -> 0.2; trace_width 1 -> 0.75
- net class PWR: clearance 0.5 -> 0.2; trace_width 0.75 -> 0.5
- rule trace_clearance: 0.5 -> 0.2
