File: AP3429-tryout.kicad_pcb (KiCad board)
At the start: 2 copper layers, 90 x 75 mm, 61 parts, among them J1 Conn_01x05, J2 Conn_01x02, U1 AP3429, U10 AMS1117-3.3, U2 AP3429, U3 AP3429, U4 AP2120N, U5 AMS1117-3.3, U6 AMS1117-3.3, U7 AMS1117-3.3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

Commit message: update,
Parts:
- added D2: LED_ORANGE, LED_SMD:LED_0805_2012Metric_Castellated, F.Cu at (2.22, 51.7)
- added R8: R103,0603, Resistor_SMD:R_0603_1608Metric_Pad1.05x0.95mm_HandSolder, F.Cu at (5.22, 51.7)
- moved D1 7.11 mm to (2.22, 42.3)
- moved R7 1.51 mm to (5.22, 42.3)
Routing:
- net GND: track 395.1 -> 413.2 mm
- net +5V: track 287.3 -> 296.7 mm
- net Net-(D2-Pad2): track 0.00 -> 3.04 mm
- net +3V3: track 111.5 -> 112.1 mm

Commit message: update,
Parts:
- added D3: LED_ORANGE, LED_SMD:LED_0805_2012Metric_Castellated, F.Cu at (2.22, 63.4)
- added R9: R102,0603, Resistor_SMD:R_0603_1608Metric_Pad1.05x0.95mm_HandSolder, F.Cu at (5.22, 63.4)
- moved C4 1.69 mm to (32.2, 18.6)
- moved TP1 1.00 mm to (78.4, 27.6)
- moved TP2 1.00 mm to (59.8, 27.6)
- moved TP3 1.00 mm to (59.8, 42.3)
- moved TP4 1.00 mm to (78.4, 42.3)
- moved TP5 1.00 mm to (59.8, 57.0)
- moved TP6 1.00 mm to (78.4, 57.0)
- turned D2 to 270 degrees
- turned R8 to 270 degrees
Routing:
- net GND: track 413.2 -> 476.1 mm
- net +3V0: track 59.4 -> 105.0 mm, vias 1 -> 4
- net +3V3: track 112.1 -> 127.8 mm
- net +5V: track 296.7 -> 311.4 mm, vias 5 -> 3
- net Net-(C15-Pad1): track 32.8 -> 25.5 mm
- net Net-(C4-Pad2): track 27.7 -> 32.0 mm
- net Net-(C27-Pad1): track 21.9 -> 25.5 mm
- net Net-(C11-Pad1): track 21.9 -> 25.4 mm
- net Net-(C21-Pad1): track 21.9 -> 25.4 mm
- net Net-(C18-Pad1): track 22.0 -> 25.5 mm
- net Net-(C24-Pad1): track 22.0 -> 25.4 mm
- net Net-(C6-Pad2): track 35.4 -> 38.6 mm
- net Net-(D3-Pad2): track 0.00 -> 3.04 mm
- net Net-(L3-Pad1): track 9.16 -> 11.2 mm
- net Net-(C5-Pad2): track 35.5 -> 37.0 mm
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- added copper zone on B.Cu, net GND
- added copper zone on F.Cu, net GND
Other:
- board text added: "3V0"
- board text added: "3V3"
- board text added: "5V"

Commit message: update,
Routing:
- net +5V: track 311.4 -> 318.8 mm
- net GND: track 476.1 -> 480.4 mm
- net Net-(C5-Pad2): track 37.0 -> 38.7 mm
Changed lines of the file:
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@@
     (thickness 1.6)
     (drawings 11)
-    (tracks 455)
+    (tracks 463)
     (zones 0)
     (modules 65)
@@
   (segment (start 57.2219 19.3331) (end 56.82 19.735) (width 0.75) (layer F.Cu) (net 8))
   (segment (start 56.82 33.4183) (end 56.82 34.45) (width 0.75) (layer F.Cu) (net 8))
-  (segment (start 17.205 57.5) (end 19.1385 59.4335) (width 0.75) (layer F.Cu) (net 8))
-  (segment (start 19.1385 59.4335) (end 39.2715 59.4335) (width 0.75) (layer F.Cu) (net 8))
-  (segment (start 39.2715 59.4335) (end 40.325 58.38) (width 0.75) (layer F.Cu) (net 8))
   (segment (start 34.8 24.9) (end 37.44 22.26) (width 0.75) (layer F.Cu) (net 8))
   (segment (start 37.44 22.26) (end 37.44 20.315) (width 0.75) (layer F.Cu) (net 8))
@@
   (segment (start 74.4754 44.7) (end 65.35 44.7) (width 0.75) (layer F.Cu) (net 8))
   (segment (start 64.95 45.1) (end 64.95 46.65) (width 0.75) (layer F.Cu) (net 8))
+  (segment (start 39.71 61.33) (end 40.325 60.715) (width 0.75) (layer F.Cu) (net 8))
+  (segment (start 18.72 61.33) (end 39.71 61.33) (width 0.75) (layer F.Cu) (net 8))
+  (segment (start 17.205 57.5) (end 17.205 59.815) (width 0.75) (layer F.Cu) (net 8))
+  (segment (start 40.325 60.715) (end 40.325 58.38) (width 0.75) (layer F.Cu) (net 8))
+  (segment (start 17.205 59.815) (end 18.72 61.33) (width 0.75) (layer F.Cu) (net 8))
   (segment (start 36.75 52.35) (end 36.75 48.9) (width 0.3) (layer F.Cu) (net 9))
   (segment (start 36.75 48.9) (end 33.35 45.5) (width 0.3) (layer F.Cu) (net 9))
@@
   (segment (start 36.75 52.35) (end 36.75 55.88) (width 0.3) (layer F.Cu) (net 9))
   (segment (start 36.75 55.88) (end 36.69 55.94) (width 0.3) (layer F.Cu) (net 9))
-  (segment (start 40.135 37.33) (end 38.315 35.51) (width 0.3) (layer F.Cu) (net 10))
-  (segment (start 43.21 37.47) (end 40.275 37.47) (width 0.3) (layer F.Cu) (net 10))
-  (segment (start 40.275 37.47) (end 40.135 37.33) (width 0.3) (layer F.Cu) (net 10))
   (segment (start 16.36 34.88) (end 16.36 31.39) (width 0.3) (layer F.Cu) (net 10))
   (segment (start 16.36 31.39) (end 18.6073 29.1427) (width 0.3) (layer F.Cu) (net 10))
   (segment (start 18.6073 29.1427) (end 31.9477 29.1427) (width 0.3) (layer F.Cu) (net 10))
   (segment (start 31.9477 29.1427) (end 38.315 35.51) (width 0.3) (layer F.Cu) (net 10))
-  (segment (start 38.525 38.94) (end 40.135 37.33) (width 0.3) (layer F.Cu) (net 10))
+  (segment (start 38.525 35.72) (end 38.315 35.51) (width 0.3) (layer F.Cu) (net 10))
+  (segment (start 38.525 38.94) (end 38.525 35.72) (width 0.3) (layer F.Cu) (net 10))
+  (segment (start 38.525 37.47) (end 38.525 38.94) (width 0.3) (layer F.Cu) (net 10))
+  (segment (start 43.21 37.47) (end 38.525 37.47) (width 0.3) (layer F.Cu) (net 10))
   (segment (start 33.055 18.565) (end 33.055 18.65) (width 0.3) (layer F.Cu) (net 11))
   (segment (start 13.95 17.34) (end 13.95 16.3797) (width 0.3) (layer F.Cu) (net 11))
@@
   (segment (start 33.055 18.565) (end 37.44 18.565) (width 0.3) (layer F.Cu) (net 11))
   (segment (start 54.12 26.4661) (end 54.12 23.76) (width 0.5) (layer F.Cu) (net 12))
-  (segment (start 53.9488 41.0712) (end 54.12 40.9) (width 0.5) (layer F.Cu) (net 12))
-  (segment (start 54.12 40.9) (end 54.12 38.475) (width 0.5) (layer F.Cu) (net 12))
-  (segment (start 52.695 42.325) (end 53.9488 41.0712) (width 0.5) (layer F.Cu) (net 12))
   (segment (start 71.315 59.635) (end 71.315 57.04) (width 0.5) (layer F.Cu) (net 12))
   (segment (start 71.315 57.04) (end 71.315 59.635) (width 0.5) (layer F.Cu) (net 12))
@@
   (segment (start 52.695 56.465) (end 54.12 55.04) (width 0.5) (layer F.Cu) (net 12))
   (segment (start 54.12 55.04) (end 54.12 53.19) (width 0.5) (layer F.Cu) (net 12))
-  (segment (start 15.455 57.5) (end 18.2409 60.2859) (width 0.5) (layer F.Cu) (net 12))
-  (segment (start 18.2409 60.2859) (end 52.0641 60.2859) (width 0.5) (layer F.Cu) (net 12))
-  (segment (start 52.0641 60.2859) (end 52.695 59.655) (width 0.5) (layer F.Cu) (net 12))
   (segment (start 52.695 59.655) (end 52.695 57.04) (width 0.5) (layer F.Cu) (net 12))
   (segment (start 15.82 52.88) (end 15.82 54.785) (width 0.5) (layer F.Cu) (net 12))
@@
   (segment (start 71.315 42.325) (end 72.74 40.9) (width 0.5) (layer F.Cu) (net 12))
   (segment (start 72.74 40.9) (end 72.74 38.475) (width 0.5) (layer F.Cu) (net 12))
-  (segment (start 52.695 27.61) (end 53.8389 26.4661) (width 0.5) (layer F.Cu) (net 12))
-  (segment (start 53.8389 26.4661) (end 54.12 26.4661) (width 0.5) (layer F.Cu) (net 12))
   (segment (start 7 15.98) (end 7 16.2791) (width 0.5) (layer B.Cu) (net 12))
   (segment (start 72.74 53.19) (end 72.74 55.615) (width 0.5) (layer F.Cu) (net 12))
@@
   (segment (start 84.15 32.1) (end 84.15 57.15) (width 0.5) (layer F.Cu) (net 12))
   (segment (start 84.15 57.15) (end 80.95 60.35) (width 0.5) (layer F.Cu) (net 12))
-  (segment (start 57.5039 29.85) (end 54.12 26.4661) (width 0.5) (layer F.Cu) (net 12))
+  (segment (start 54.12 27.61) (end 54.12 26.4661) (width 0.5) (layer F.Cu) (net 12))
+  (segment (start 52.695 27.61) (end 54.12 27.61) (width 0.5) (layer F.Cu) (net 12))
+  (segment (start 54.12 27.58) (end 54.12 26.4661) (width 0.5) (layer F.Cu) (net 12))
+  (segment (start 56.39 29.85) (end 54.12 27.58) (width 0.5) (layer F.Cu) (net 12))
   (segment (start 64.5883 31.9125) (end 62.5258 29.85) (width 0.5) (layer F.Cu) (net 12))
-  (segment (start 62.5258 29.85) (end 57.5039 29.85) (width 0.5) (layer F.Cu) (net 12))
-  (segment (start 57.3276 44.45) (end 53.9488 41.0712) (width 0.5) (layer F.Cu) (net 12))
+  (segment (start 62.5258 29.85) (end 56.39 29.85) (width 0.5) (layer F.Cu) (net 12))
+  (segment (start 52.695 42.325) (end 53.9488 42.325) (width 0.5) (layer F.Cu) (net 12))
+  (segment (start 54.12 42.1538) (end 53.9488 42.325) (width 0.5) (layer F.Cu) (net 12))
+  (segment (start 54.12 39.49) (end 54.12 38.475) (width 0.5) (layer F.Cu) (net 12))
   (segment (start 64.5883 43.55) (end 63.6883 44.45) (width 0.5) (layer F.Cu) (net 12))
-  (segment (start 63.6883 44.45) (end 57.3276 44.45) (width 0.5) (layer F.Cu) (net 12))
+  (segment (start 58.63 44.45) (end 55.42 44.45) (width 0.5) (layer F.Cu) (net 12))
+  (segment (start 63.6883 44.45) (end 58.63 44.45) (width 0.5) (layer F.Cu) (net 12))
+  (segment (start 54.12 43.15) (end 54.12 41.58) (width 0.5) (layer F.Cu) (net 12))
+  (segment (start 55.42 44.45) (end 54.12 43.15) (width 0.5) (layer F.Cu) (net 12))
+  (segment (start 54.12 39.49) (end 54.12 41.58) (width 0.5) (layer F.Cu) (net 12))
+  (segment (start 54.12 41.58) (end 54.12 42.1538) (width 0.5) (layer F.Cu) (net 12))
+  (segment (start 18.69 63.81) (end 48.54 63.81) (width 0.5) (layer F.Cu) (net 12))
+  (segment (start 15.455 57.5) (end 15.455 60.575) (width 0.5) (layer F.Cu) (net 12))
+  (segment (start 48.54 63.81) (end 52.695 59.655) (width 0.5) (layer F.Cu) (net 12))
+  (segment (start 15.455 60.575) (end 18.69 63.81) (width 0.5) (layer F.Cu) (net 12))
   (segment (start 12.1018 33.9982) (end 10.56 35.54) (width 0.5) (layer B.Cu) (net 13))
   (segment (start 10.56 35.54) (end 7 35.54) (width 0.5) (layer B.Cu) (net 13))
