File: tryout/1V2_tryout/1V2_tryout.sch (KiCad schematic (older format))
At the start: 7 parts

Commit message: update,
Parts:
- gave numbers to parts that had none: 7
Changed lines of the file:
@@
 EESchema Schematic File Version 4
-LIBS:AP3429-tryout-cache
+LIBS:1V2_tryout-cache
 EELAYER 26 0
 EELAYER END
@@
 $EndDescr
 $Comp
-L taobao-components:AP3429 U?
+L taobao-components:AP3429 U1
 U 1 1 5C0388AE
 P 5250 3550
-F 0 "U?" H 5250 4165 50  0000 C CNN
+F 0 "U1" H 5250 4165 50  0000 C CNN
 F 1 "AP3429" H 5250 4074 50  0000 C CNN
 F 2 "Package_TO_SOT_SMD:TSOT-23-5" H 5200 3450 50  0001 C CNN
@@
 $EndComp
 $Comp
-L power:+5V #PWR?
+L power:+5V #PWR0101
 U 1 1 5C038C0E
 P 3650 3000
-F 0 "#PWR?" H 3650 2850 50  0001 C CNN
+F 0 "#PWR0101" H 3650 2850 50  0001 C CNN
 F 1 "+5V" H 3665 3173 50  0000 C CNN
 F 2 "" H 3650 3000 50  0001 C CNN
@@
 	3650 3300 3650 3750
 $Comp
-L power:GND #PWR?
+L power:GND #PWR0102
 U 1 1 5C038E38
 P 3650 4500
-F 0 "#PWR?" H 3650 4250 50  0001 C CNN
+F 0 "#PWR0102" H 3650 4250 50  0001 C CNN
 F 1 "GND" H 3655 4327 50  0000 C CNN
 F 2 "" H 3650 4500 50  0001 C CNN
@@
 	4200 3300 3650 3300
 $Comp
-L taobao-r:R304,0603 R?
+L taobao-r:R304,0603 R1
 U 1 1 5C03943C
 P 7300 3450
-F 0 "R?" H 7359 3496 50  0000 L CNN
+F 0 "R1" H 7359 3496 50  0000 L CNN
 F 1 "R304,0603" H 7359 3405 50  0000 L CNN
 F 2 "Resistor_SMD:R_0603_1608Metric_Pad1.05x0.95mm_HandSolder" H 7300 3450 50  0001 C CNN
@@
 $EndComp
 $Comp
-L taobao-r:R304,0603 R?
+L taobao-r:R304,0603 R2
 U 1 1 5C0394B6
 P 7300 4150
-F 0 "R?" H 7359 4196 50  0000 L CNN
+F 0 "R2" H 7359 4196 50  0000 L CNN
 F 1 "R304,0603" H 7359 4105 50  0000 L CNN
 F 2 "Resistor_SMD:R_0603_1608Metric_Pad1.05x0.95mm_HandSolder" H 7300 4150 50  0001 C CNN
@@
 	7300 3750 7300 4050
 $Comp
-L power:+1V2 #PWR?
+L power:+1V2 #PWR0103
 U 1 1 5C03A34B
 P 8200 3250
-F 0 "#PWR?" H 8200 3100 50  0001 C CNN
+F 0 "#PWR0103" H 8200 3100 50  0001 C CNN
 F 1 "+1V2" H 8215 3423 50  0000 C CNN
 F 2 "" H 8200 3250 50  0001 C CNN
@@
 Connection ~ 7300 4400
 $Comp
-L taobao-c:C22pf,0603 C?
+L taobao-c:C22pf,0603 C2
 U 1 1 5C06221C
 P 6850 3550
-F 0 "C?" H 6942 3596 50  0000 L CNN
+F 0 "C2" H 6942 3596 50  0000 L CNN
 F 1 "C22pf,0603" H 6942 3505 50  0000 L CNN
 F 2 "Capacitor_SMD:C_0603_1608Metric_Pad1.05x0.95mm_HandSolder" H 6850 3550 50  0001 C CNN
@@
 $EndComp
 $Comp
-L taobao-c:C226,6.3v,0603 C?
+L taobao-c:C226,6.3v,0603 C1
 U 1 1 5C03CE8D
 P 3650 3850
-F 0 "C?" H 3742 3896 50  0000 L CNN
+F 0 "C1" H 3742 3896 50  0000 L CNN
 F 1 "C226,6.3v,0603" H 3742 3805 50  0000 L CNN
 F 2 "Capacitor_SMD:C_0603_1608Metric_Pad1.05x0.95mm_HandSolder" H 3650 3850 50  0001 C CNN
@@
 $EndComp
 $Comp
-L taobao-c:C226,6.3v,0603 C?
+L taobao-c:C226,6.3v,0603 C3
 U 1 1 5C03CF94
 P 8200 3650
-F 0 "C?" H 8292 3696 50  0000 L CNN
+F 0 "C3" H 8292 3696 50  0000 L CNN
 F 1 "C226,6.3v,0603" H 8292 3605 50  0000 L CNN
 F 2 "Capacitor_SMD:C_0603_1608Metric_Pad1.05x0.95mm_HandSolder" H 8200 3650 50  0001 C CNN
@@
 $EndComp
 $Comp
-L taobao-l:L_2.2uH,1210 L?
+L taobao-l:L_2.2uH,1210 L1
 U 1 1 5C0651A2
 P 6400 3300
-F 0 "L?" V 6600 3300 50  0000 C CNN
+F 0 "L1" V 6600 3300 50  0000 C CNN
 F 1 "L_2.2uH,1210" V 6500 3300 50  0000 C CNN
 F 2 "Inductor_SMD:L_1210_3225Metric_Pad1.42x2.65mm_HandSolder" H 6400 3300 50  0001 C CNN
