File: tryout/1V2_tryout/1V2_tryout.kicad_pcb (KiCad board)
At the start: 2 copper layers, 7 parts, among them U1 AP3429

Commit message: update,
Parts:
- moved C1 10.8 mm to (14.0, 26.0), turned to 0 degrees
- moved L1 6.08 mm to (18.0, 22.0), turned to 90 degrees
- moved C2 5.00 mm to (25.0, 22.0)
- moved R1 5.00 mm to (23.0, 22.0)
- moved R2 5.00 mm to (27.0, 22.0)
- moved C3 3.00 mm to (21.0, 22.0), turned to 270 degrees
Routing:
- net +5V: track 16.5 -> 6.80 mm, vias 2 -> 0
- net Net-(C2-Pad2): track 9.77 -> 15.7 mm, vias 2 -> 0
- net GND: track 13.5 -> 16.9 mm, vias 2 -> 0
- net Net-(L1-Pad1): track 4.92 -> 4.30 mm
Other:
- board outline added: 24 x 13 mm
