File: tryout/1V8_tryout/1V8_tryout.sch (KiCad schematic (older format))
At the start: 7 parts

Commit message: update,
Parts:
- gave numbers to parts that had none: 7
Changed lines of the file:
@@
 EESchema Schematic File Version 4
-LIBS:AP3429-tryout-cache
+LIBS:1V8_tryout-cache
 EELAYER 26 0
 EELAYER END
@@
 $EndDescr
 $Comp
-L taobao-components:AP3429 U?
+L taobao-components:AP3429 U1
 U 1 1 5C03B1FE
 P 3550 3700
-F 0 "U?" H 3550 4315 50  0000 C CNN
+F 0 "U1" H 3550 4315 50  0000 C CNN
 F 1 "AP3429" H 3550 4224 50  0000 C CNN
 F 2 "Package_TO_SOT_SMD:TSOT-23-5" H 3500 3600 50  0001 C CNN
@@
 $EndComp
 $Comp
-L power:+5V #PWR?
+L power:+5V #PWR0101
 U 1 1 5C03B204
 P 1950 3150
-F 0 "#PWR?" H 1950 3000 50  0001 C CNN
+F 0 "#PWR0101" H 1950 3000 50  0001 C CNN
 F 1 "+5V" H 1965 3323 50  0000 C CNN
 F 2 "" H 1950 3150 50  0001 C CNN
@@
 	1950 3450 1950 3900
 $Comp
-L power:GND #PWR?
+L power:GND #PWR0102
 U 1 1 5C03B214
 P 1950 4650
-F 0 "#PWR?" H 1950 4400 50  0001 C CNN
+F 0 "#PWR0102" H 1950 4400 50  0001 C CNN
 F 1 "GND" H 1955 4477 50  0000 C CNN
 F 2 "" H 1950 4650 50  0001 C CNN
@@
 	2500 3450 1950 3450
 $Comp
-L taobao-r:R304,0603 R?
+L taobao-r:R304,0603 R1
 U 1 1 5C03B22A
 P 5600 3600
-F 0 "R?" H 5659 3646 50  0000 L CNN
+F 0 "R1" H 5659 3646 50  0000 L CNN
 F 1 "R304,0603" H 5659 3555 50  0000 L CNN
 F 2 "Resistor_SMD:R_0603_1608Metric_Pad1.05x0.95mm_HandSolder" H 5600 3600 50  0001 C CNN
@@
 Connection ~ 5600 4550
 $Comp
-L taobao-r:R154,0603 R?
+L taobao-r:R154,0603 R2
 U 1 1 5C03DAA8
 P 5600 4300
-F 0 "R?" H 5659 4346 50  0000 L CNN
+F 0 "R2" H 5659 4346 50  0000 L CNN
 F 1 "R154,0603" H 5659 4255 50  0000 L CNN
 F 2 "Resistor_SMD:R_0603_1608Metric_Pad1.05x0.95mm_HandSolder" H 5600 4300 50  0001 C CNN
@@
 $EndComp
 $Comp
-L power:+1V8 #PWR?
+L power:+1V8 #PWR0103
 U 1 1 5C03DEFC
 P 6500 3400
-F 0 "#PWR?" H 6500 3250 50  0001 C CNN
+F 0 "#PWR0103" H 6500 3250 50  0001 C CNN
 F 1 "+1V8" H 6515 3573 50  0000 C CNN
 F 2 "" H 6500 3400 50  0001 C CNN
@@
 $EndComp
 $Comp
-L taobao-c:C22pf,0603 C?
+L taobao-c:C22pf,0603 C2
 U 1 1 5C0621B0
 P 5150 3700
-F 0 "C?" H 5242 3746 50  0000 L CNN
+F 0 "C2" H 5242 3746 50  0000 L CNN
 F 1 "C22pf,0603" H 5242 3655 50  0000 L CNN
 F 2 "Capacitor_SMD:C_0603_1608Metric_Pad1.05x0.95mm_HandSolder" H 5150 3700 50  0001 C CNN
@@
 $EndComp
 $Comp
-L taobao-c:C226,6.3v,0603 C?
+L taobao-c:C226,6.3v,0603 C3
 U 1 1 5C03D10B
 P 6500 3800
-F 0 "C?" H 6592 3846 50  0000 L CNN
+F 0 "C3" H 6592 3846 50  0000 L CNN
 F 1 "C226,6.3v,0603" H 6592 3755 50  0000 L CNN
 F 2 "Capacitor_SMD:C_0603_1608Metric_Pad1.05x0.95mm_HandSolder" H 6500 3800 50  0001 C CNN
@@
 $EndComp
 $Comp
-L taobao-c:C226,6.3v,0603 C?
+L taobao-c:C226,6.3v,0603 C1
 U 1 1 5C03D1E9
 P 1950 4000
-F 0 "C?" H 2042 4046 50  0000 L CNN
+F 0 "C1" H 2042 4046 50  0000 L CNN
 F 1 "C226,6.3v,0603" H 2042 3955 50  0000 L CNN
 F 2 "Capacitor_SMD:C_0603_1608Metric_Pad1.05x0.95mm_HandSolder" H 1950 4000 50  0001 C CNN
@@
 $EndComp
 $Comp
-L taobao-l:L_2.2uH,1210 L?
+L taobao-l:L_2.2uH,1210 L1
 U 1 1 5C0652FE
 P 4700 3450
-F 0 "L?" V 4900 3450 50  0000 C CNN
+F 0 "L1" V 4900 3450 50  0000 C CNN
 F 1 "L_2.2uH,1210" V 4800 3450 50  0000 C CNN
 F 2 "Inductor_SMD:L_1210_3225Metric_Pad1.42x2.65mm_HandSolder" H 4700 3450 50  0001 C CNN
