File: tryout/3V3_tryout/3V3_tryout.sch (KiCad schematic (older format))
At the start: 9 parts

Commit message: update,
Parts:
- gave numbers to parts that had none: 9
Changed lines of the file:
@@
 EESchema Schematic File Version 4
-LIBS:AP3429-tryout-cache
+LIBS:3V3_tryout-cache
 EELAYER 26 0
 EELAYER END
@@
 $EndDescr
 $Comp
-L taobao-components:AP3429 U?
+L taobao-components:AP3429 U1
 U 1 1 5C03BEFC
 P 3400 2400
-F 0 "U?" H 3400 3015 50  0000 C CNN
+F 0 "U1" H 3400 3015 50  0000 C CNN
 F 1 "AP3429" H 3400 2924 50  0000 C CNN
 F 2 "Package_TO_SOT_SMD:TSOT-23-5" H 3350 2300 50  0001 C CNN
@@
 $EndComp
 $Comp
-L power:+5V #PWR?
+L power:+5V #PWR0101
 U 1 1 5C03BF02
 P 1800 1850
-F 0 "#PWR?" H 1800 1700 50  0001 C CNN
+F 0 "#PWR0101" H 1800 1700 50  0001 C CNN
 F 1 "+5V" H 1815 2023 50  0000 C CNN
 F 2 "" H 1800 1850 50  0001 C CNN
@@
 	1800 2150 1800 2650
 $Comp
-L power:GND #PWR?
+L power:GND #PWR0102
 U 1 1 5C03BF12
 P 1800 3350
-F 0 "#PWR?" H 1800 3100 50  0001 C CNN
+F 0 "#PWR0102" H 1800 3100 50  0001 C CNN
 F 1 "GND" H 1805 3177 50  0000 C CNN
 F 2 "" H 1800 3350 50  0001 C CNN
@@
 Connection ~ 5450 3250
 $Comp
-L power:+3V3 #PWR?
+L power:+3V3 #PWR0103
 U 1 1 5C03E213
 P 6350 2100
-F 0 "#PWR?" H 6350 1950 50  0001 C CNN
+F 0 "#PWR0103" H 6350 1950 50  0001 C CNN
 F 1 "+3V3" H 6365 2273 50  0000 C CNN
 F 2 "" H 6350 2100 50  0001 C CNN
@@
 $EndComp
 $Comp
-L taobao-r:R184,0603 R?
+L taobao-r:R184,0603 R2
 U 1 1 5C042158
 P 5450 3000
-F 0 "R?" H 5509 3046 50  0000 L CNN
+F 0 "R2" H 5509 3046 50  0000 L CNN
 F 1 "R184,0603" H 5509 2955 50  0000 L CNN
 F 2 "Resistor_SMD:R_0603_1608Metric_Pad1.05x0.95mm_HandSolder" H 5450 3000 50  0001 C CNN
@@
 $EndComp
 $Comp
-L taobao-led:LED_ORANGE D?
+L taobao-led:LED_ORANGE D1
 U 1 1 5C042628
 P 8650 4100
-F 0 "D?" V 8696 4032 50  0000 R CNN
+F 0 "D1" V 8696 4032 50  0000 R CNN
 F 1 "LED_ORANGE" V 8605 4032 50  0000 R CNN
 F 2 "LED_SMD:LED_0805_2012Metric_Castellated" V 8650 4100 50  0001 C CNN
@@
 $EndComp
 $Comp
-L taobao-r:R102,0603 R?
+L taobao-r:R102,0603 R3
 U 1 1 5C04282E
 P 8650 3750
-F 0 "R?" H 8709 3796 50  0000 L CNN
+F 0 "R3" H 8709 3796 50  0000 L CNN
 F 1 "R102,0603" H 8709 3705 50  0000 L CNN
 F 2 "Resistor_SMD:R_0603_1608Metric_Pad1.05x0.95mm_HandSolder" H 8650 3750 50  0001 C CNN
@@
 	8650 4200 8650 4500
 $Comp
-L taobao-r:R824,0603 R?
+L taobao-r:R824,0603 R1
 U 1 1 5C052FAD
 P 5450 2350
-F 0 "R?" H 5509 2396 50  0000 L CNN
+F 0 "R1" H 5509 2396 50  0000 L CNN
 F 1 "R824,0603" H 5509 2305 50  0000 L CNN
 F 2 "Resistor_SMD:R_0603_1608Metric_Pad1.05x0.95mm_HandSolder" H 5450 2350 50  0001 C CNN
@@
 $EndComp
 $Comp
-L taobao-c:C22pf,0603 C?
+L taobao-c:C22pf,0603 C2
 U 1 1 5C061E10
 P 5000 2400
-F 0 "C?" H 5092 2446 50  0000 L CNN
+F 0 "C2" H 5092 2446 50  0000 L CNN
 F 1 "C22pf,0603" H 5092 2355 50  0000 L CNN
 F 2 "Capacitor_SMD:C_0603_1608Metric_Pad1.05x0.95mm_HandSolder" H 5000 2400 50  0001 C CNN
@@
 $EndComp
 $Comp
-L taobao-c:C226,6.3v,0603 C?
+L taobao-c:C226,6.3v,0603 C3
 U 1 1 5C03D3A0
 P 6350 2500
-F 0 "C?" H 6442 2546 50  0000 L CNN
+F 0 "C3" H 6442 2546 50  0000 L CNN
 F 1 "C226,6.3v,0603" H 6442 2455 50  0000 L CNN
 F 2 "Capacitor_SMD:C_0603_1608Metric_Pad1.05x0.95mm_HandSolder" H 6350 2500 50  0001 C CNN
@@
 $EndComp
 $Comp
-L taobao-c:C226,6.3v,0603 C?
+L taobao-c:C226,6.3v,0603 C1
 U 1 1 5C03D426
 P 1800 2750
-F 0 "C?" H 1892 2796 50  0000 L CNN
+F 0 "C1" H 1892 2796 50  0000 L CNN
 F 1 "C226,6.3v,0603" H 1892 2705 50  0000 L CNN
 F 2 "Capacitor_SMD:C_0603_1608Metric_Pad1.05x0.95mm_HandSolder" H 1800 2750 50  0001 C CNN
@@
 $EndComp
 $Comp
-L taobao-l:L_2.2uH,1210 L?
+L taobao-l:L_2.2uH,1210 L1
 U 1 1 5C0655CA
 P 4550 2150
-F 0 "L?" V 4600 1900 50  0000 R CNN
+F 0 "L1" V 4600 1900 50  0000 R CNN
 F 1 "L_2.2uH,1210" V 4550 1900 50  0000 R CNN
 F 2 "Inductor_SMD:L_1210_3225Metric_Pad1.42x2.65mm_HandSolder" H 4550 2150 50  0001 C CNN
@@
 	5450 3250 6350 3250
 $Comp
-L power:+3V3 #PWR?
+L power:+3V3 #PWR0104
 U 1 1 5C078F9C
 P 8650 3400
-F 0 "#PWR?" H 8650 3250 50  0001 C CNN
+F 0 "#PWR0104" H 8650 3250 50  0001 C CNN
 F 1 "+3V3" H 8665 3573 50  0000 C CNN
 F 2 "" H 8650 3400 50  0001 C CNN
@@
 $EndComp
 $Comp
-L power:GND #PWR?
+L power:GND #PWR0105
 U 1 1 5C079499
 P 8650 4500
-F 0 "#PWR?" H 8650 4250 50  0001 C CNN
+F 0 "#PWR0105" H 8650 4250 50  0001 C CNN
 F 1 "GND" H 8655 4327 50  0000 C CNN
 F 2 "" H 8650 4500 50  0001 C CNN
